File: chevron_esp.kicad_sch (KiCad schematic)
At the start: 20 parts, among them J1 282837-4, K1 SRD-05VDC-SL-C, K2 SRD-05VDC-SL-C, K3 SRD-05VDC-SL-C, P1 282837-2, Q1 PN2222A, Q2 PN2222A, Q3 PN2222A, SW1 1825057-2, U1 ESP32-DEVKIT-V1, U2 RA-02_LORA

Commit message: chevron esp v1.0
Parts:
- renumbered R11 to R1, R12 to R2, R13 to R3, R14 to R4, R15 to R5, R16 to R6
Other:
- moved on the sheet: D13, D14, D15, J1, K1, K2, K3, P1, Q1, Q2, Q3, R1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
